Commit message: float depth hold PID tuned

File: oasis_auv_stonefish/description/oasis_auv.scn.xacro (robot description, xacro)
@@ -30,24 +30,30 @@
                     <cg xyz="0.565 0.0 0.00" rpy="0.0 0.0 0.0"/>
                 </external_part>
-                <internal_part name="lumsum_body" type="cylinder" physics="surface" buoyant="true">
+                <internal_part name="lumsum_buoyancy" type="cylinder" physics="surface" buoyant="true">
                     <dimensions radius="0.08" height="1.22"/>
-                    <origin rpy="0.0 -1.571 0.0" xyz="0.5 0.0 0.0"/>
+                    <origin rpy="0.0 -1.571 0.0" xyz="0.6 0.0 -0.0025"/>
                     <material name="Neutral"/>
-                    <mass value="21.0"/>
+                    <mass value="0.001"/>
                     <look name="grey"/>
-                    <!-- <compound_transform rpy= "0.0 0.0 0.0" xyz="0.9 0 0.057"/> -->
-                    <!-- <compound_transform rpy= "0.0 0.0 0.0" xyz="0.847 0 0.057"/> -->
                     <compound_transform rpy= "0.0 0.0 0.0" xyz="0.0 0 0.0"/>
                 </internal_part>
-                <internal_part name="Foam" type="box" physics="surface" buoyant="true">
+                <internal_part name="lumsum_weight" type="cylinder" physics="surface" buoyant="false">
+                    <dimensions radius="0.08" height="0.5"/>
+                    <origin rpy="0.0 -1.571 0.0" xyz="0.57 0.0 0.0025"/>
+                    <material name="Stainless_steel"/>
+                    <mass value="22.2"/>
+                    <look name="red"/>
+                    <compound_transform rpy= "0.0 0.0 0.0" xyz="0.0 0 0.0"/>
+                </internal_part>
+                <internal_part name="Weight" type="box" physics="surface" buoyant="true">
                     <dimensions xyz="0.23 0.058 0.042"/>
                     <origin rpy="0.0 0.0 0.0" xyz="0.0 0.0 0.0"/>
                     <material name="Stainless_steel"/>
-                    <mass value="4.0"/>
-                    <look name="grey"/>
-                    <!-- <compound_transform rpy= "0.0 0.0 0.0" xyz="0.9 0 0.057"/> -->
+                    <mass value="3.0"/>
+                    <look name="yellow"/>
+                    <!-- forward position -->
                     <!-- <compound_transform rpy= "0.0 0.0 0.0" xyz="0.847 0 0.057"/> -->
-                    <compound_transform rpy= "0.0 0.0 0.0" xyz="0.5 0 0.057"/>
-                    <!-- <compound_transform rpy= "0.0 0.0 0.0" xyz="0.347 0 0.057"/> -->
+                    <!-- backward position -->
+                    <compound_transform rpy= "0.0 0.0 0.0" xyz="0.347 0 0.057"/>
                 </internal_part>
                 <external_part name="ThrusterDuctSurge" type="model" physics="surface" buoyant="true">
