Commit message: tested direct control behavior

File: oasis_auv_description/urdf/base.urdf.xacro (robot description, xacro)
@@ -3,5 +3,5 @@
     <link name="base_link">
         <visual>
-            <origin xyz="0.0 -0.63 -0.57" rpy="0.0 0.0 1.5707963"/>
+            <origin xyz="-0.5 0.0 0.184" rpy="3.1415926 0.0 3.1415926"/>
             <geometry>
                 <mesh filename="package://oasis_auv_description/mesh/oasis_auv.obj" scale="1 1 1"/>
@@ -17,5 +17,5 @@
     <link name="imu"/>
     <joint name="imu_joint" type="fixed">
-        <origin xyz="0.0 0.0 0.0" rpy="0.0 0.0 0.0"/>
+        <origin xyz="-0.3 0.0 0.092" rpy="0.0 0.0 0.0"/>
         <parent link="base_link"/>
         <child link="imu"/>
@@ -23,5 +23,5 @@
     <link name="imu_sf"/>
     <joint name="imu__sf_joint" type="fixed">
-        <origin xyz="0.0 0.0 0.0" rpy="0.0 0.0 0.0"/>
+        <origin xyz="-0.3 0.0 0.092" rpy="3.1415926 0.0 0.0"/>
         <parent link="base_link"/>
         <child link="imu_sf"/>
@@ -29,5 +29,5 @@
     <link name="dvl"/>
     <joint name="dvl_joint" type="fixed">
-        <origin xyz="-0.22 0.0 -0.08" rpy="3.1415926 0.0 0.0"/>
+        <origin xyz="-0.3 0.0 0.092" rpy="0.0 0.0 0.0"/>
         <parent link="base_link"/>
         <child link="dvl"/>
@@ -35,5 +35,5 @@
      <link name="dvl_sf"/>
     <joint name="dvl_sf_joint" type="fixed">
-        <origin xyz="-0.22 0.0 -0.08" rpy="0.0 0.0 0.0"/>
+        <origin xyz="-0.3 0.0 0.092" rpy="3.1415926 0.0 0.0"/>
         <parent link="base_link"/>
         <child link="dvl_sf"/>
@@ -47,5 +47,5 @@
     <link name="pressure"/>
     <joint name="pressure_joint" type="fixed">
-        <origin xyz="-0.25 0.0 0.05" rpy="3.1415926 0.0 0.0"/>
+        <origin xyz="-0.2 0.0 0.091" rpy="3.1415926 0.0 0.0"/>
         <parent link="base_link"/>
         <child link="pressure"/>
@@ -54,5 +54,5 @@
     <link name="surge_thruster_link"/>
     <joint name="surge_thruster_joint" type="fixed">
-        <origin xyz="-0.68 0.0 0.0" rpy="0.0 0.0 0.0"/>
+        <origin xyz="-0.5 0.0 0.0" rpy="0.0 0.0 0.0"/>
         <parent link="base_link"/>
         <child link="surge_thruster_link"/>
@@ -60,5 +60,5 @@
     <link name="heave_bow_thruster_link"/>
     <joint name="heave_bow_thruster_joint" type="fixed">
-        <origin xyz="0.38 0.0 0.0" rpy="0.0 1.57079632679 0.0"/>
+        <origin xyz="0.7674 0.0 0.03" rpy="0.0 1.57079632679 0.0"/>
         <parent link="base_link"/>
         <child link="heave_bow_thruster_link"/>
@@ -66,5 +66,5 @@
     <link name="sway_thruster_link"/>
     <joint name="sway_thruster_joint" type="fixed">
-        <origin xyz="0.48 0.0 0.0" rpy="0.0 0.0 -1.57079632679"/>
+        <origin xyz="-0.27 0.0 -0.038" rpy="0.0 0.0 -1.57079632679"/>
         <parent link="base_link"/>
         <child link="sway_thruster_link"/>

File: oasis_auv_stonefish/description/oasis_auv.scn.xacro (robot description, xacro)
@@ -103,20 +103,20 @@
             <sensor name="pressure" type="pressure" rate="5.0">
                 <link name="Base"/>
-                <origin rpy="0.0 0.0 0.0" xyz="0.1 0.0 0.0"/>
-                <noise pressure="2.0"/>
+                <origin rpy="0.0 0.0 0.0" xyz="0.1 0.0 -0.091"/>
+                <noise pressure="0.0"/>
                 <ros_publisher topic="/${robot_name}/pressure"/>
             </sensor>
             <sensor name="dvl_sf" type="dvl" rate="5.0">
                 <link name="Base"/>
-                <origin rpy="3.1415926 0.0 0.0" xyz="0.65 0.0 0.092"/>
+                <origin rpy="0.0 0.0 0.0" xyz="0.1 0.0 -0.092"/>
                 <specs beam_angle="30.0"/>
                 <range velocity="9.0 9.0 9.0" altitude_min="0.2" altitude_max="200.0"/>
-                <noise velocity="0.015" altitude="0.001"/>
+                <noise velocity="0.0" altitude="0.00"/>
                 <ros_publisher topic="/${robot_name}/dvl/twist" altitude_topic="/${robot_name}/dvl/altitude"/>
             </sensor>
             <sensor name="imu_sf" type="imu" rate="20.0">
                 <link name="Base"/>
-                <origin rpy="3.1415926 0.0 0.0" xyz="0.65 0.0 0.092"/>
-                <noise angle="0.01 0.01 0.05" angular_velocity="0.05" yaw_drift="0.001" linear_acceleration="0.1"/>
+                <origin rpy="3.1415926 0.0 0.0" xyz="0.1 0.0 -0.092"/>
+                <noise angle="0.00 0.00 0.00" angular_velocity="0.00" yaw_drift="0.000" linear_acceleration="0.0"/>
                 <ros_publisher topic="/${robot_name}/imu/stonefish/data"/>
             </sensor>

Commit message: fixed imu rotation

File: oasis_auv_description/urdf/base.urdf.xacro (robot description, xacro)
@@ -23,5 +23,5 @@
     <link name="imu_sf"/>
     <joint name="imu__sf_joint" type="fixed">
-        <origin xyz="-0.3 0.0 0.092" rpy="3.1415926 0.0 0.0"/>
+        <origin xyz="-0.3 0.0 0.092" rpy="0.0 0.0 0.0"/>
         <parent link="base_link"/>
         <child link="imu_sf"/>
@@ -66,5 +66,5 @@
     <link name="sway_thruster_link"/>
     <joint name="sway_thruster_joint" type="fixed">
-        <origin xyz="-0.27 0.0 -0.038" rpy="0.0 0.0 -1.57079632679"/>
+        <origin xyz="-0.27 0.0 0.0" rpy="0.0 0.0 -1.57079632679"/>
         <parent link="base_link"/>
         <child link="sway_thruster_link"/>

File: oasis_auv_stonefish/description/oasis_auv.scn.xacro (robot description, xacro)
@@ -37,6 +37,6 @@
                     <look name="grey"/>
                     <!-- <compound_transform rpy= "0.0 0.0 0.0" xyz="0.9 0 0.057"/> -->
-                    <!-- <compound_transform rpy= "0.0 0.0 0.0" xyz="0.847 0 0.057"/> -->
-                    <compound_transform rpy= "0.0 0.0 0.0" xyz="0.347 0 0.057"/>
+                    <compound_transform rpy= "0.0 0.0 0.0" xyz="0.847 0 0.057"/>
+                    <!-- <compound_transform rpy= "0.0 0.0 0.0" xyz="0.347 0 0.057"/> -->
                 </internal_part>
                 <external_part name="ThrusterDuctSurge" type="model" physics="surface" buoyant="true">
@@ -69,5 +69,5 @@
             <actuator name="ThrusterSway" type="thruster">
                 <link name="Base"/>
-                <origin rpy="0.0 0.0 1.5707963" xyz="0.07 0.0 0.038"/>
+                <origin rpy="0.0 0.0 1.5707963" xyz="0.07 0.0 0.0"/>
                 <specs thrust_coeff="0.4315" thrust_coeff_backward="0.3404" torque_coeff="0.01" max_rpm="3000.0"/>
                 <propeller diameter="0.08" right="true">
@@ -78,4 +78,5 @@
                 <ros_subscriber topic="/${robot_name}/control/thruster/sway"/>
             </actuator>
+<!--
             <actuator name="ThrusterHeaveBow" type="thruster">
                 <link name="Base"/>
@@ -100,5 +101,5 @@
                 </propeller>
                 <ros_subscriber topic="/${robot_name}/control/thruster/surge"/>
-            </actuator>
+            </actuator> -->
             <sensor name="pressure" type="pressure" rate="5.0">
                 <link name="Base"/>

Commit message: heading control validated, PID needs to be tuned

File: oasis_auv_description/urdf/base.urdf.xacro (robot description, xacro)
@@ -66,5 +66,6 @@
     <link name="sway_thruster_link"/>
     <joint name="sway_thruster_joint" type="fixed">
-        <origin xyz="-0.27 0.0 0.0" rpy="0.0 0.0 -1.57079632679"/>
+        <origin xyz="-0.27 0.0 -0.038" rpy="0.0 0.0 -1.57079632679"/>
+        <!-- <origin xyz="-0.27 0.0 -0.0" rpy="0.0 0.0 -1.57079632679"/> -->
         <parent link="base_link"/>
         <child link="sway_thruster_link"/>

File: oasis_auv_stonefish/description/oasis_auv.scn.xacro (robot description, xacro)
@@ -69,5 +69,6 @@
             <actuator name="ThrusterSway" type="thruster">
                 <link name="Base"/>
-                <origin rpy="0.0 0.0 1.5707963" xyz="0.07 0.0 0.0"/>
+                <origin rpy="0.0 0.0 1.5707963" xyz="0.07 0.0 0.038"/>
+                <!-- <origin rpy="0.0 0.0 1.5707963" xyz="0.07 0.0 0.0"/> -->
                 <specs thrust_coeff="0.4315" thrust_coeff_backward="0.3404" torque_coeff="0.01" max_rpm="3000.0"/>
                 <propeller diameter="0.08" right="true">
@@ -78,5 +79,4 @@
                 <ros_subscriber topic="/${robot_name}/control/thruster/sway"/>
             </actuator>
-<!--
             <actuator name="ThrusterHeaveBow" type="thruster">
                 <link name="Base"/>
@@ -101,5 +101,5 @@
                 </propeller>
                 <ros_subscriber topic="/${robot_name}/control/thruster/surge"/>
-            </actuator> -->
+            </actuator>
             <sensor name="pressure" type="pressure" rate="5.0">
                 <link name="Base"/>

File: oasis_auv_stonefish/scenarios/under_ice.scn.xacro (robot description, xacro)
@@ -30,5 +30,5 @@
         </atmosphere>
     </environment>
-    <static name="Ice" type="model">
+    <!-- <static name="Ice" type="model">
         <physical>
             <mesh filename="ice_cover.obj" scale="1.0" convex="false"/>
@@ -42,4 +42,4 @@
         <look name="ice"/>
         <world_transform xyz="0.0 0.0 0.0" rpy="0.0 0.0 0.0"/>
-    </static>
+    </static> -->
 </scenario>
