Commit message: added one more thruster and adjusted the weight

File: oasis_auv_description/urdf/base_sf.urdf.xacro (robot description, xacro)
@@ -11,5 +11,5 @@
     <link name="cg_link"/>
     <joint name="cg_joint" type="fixed">
-        <origin xyz="0.0 0.0 0.0" rpy="3.1415926 0.0 0.0"/>
+        <origin xyz="0.3374 0.0 0.0" rpy="3.1415926 0.0 0.0"/>
         <parent link="base_link"/>
         <child link="cg_link"/>
@@ -64,8 +64,14 @@
         <child link="heave_bow_thruster_link"/>
     </joint>
+    <link name="heave_stern_thruster_link"/>
+    <joint name="heave_stern_thruster_joint" type="fixed">
+        <origin xyz="-0.0926 0.0 0.03" rpy="0.0 1.57079632679 0.0"/>
+        <parent link="base_link"/>
+        <child link="heave_stern_thruster_link"/>
+    </joint>
     <link name="sway_thruster_link"/>
     <joint name="sway_thruster_joint" type="fixed">
-        <origin xyz="-0.27 0.0 -0.038" rpy="0.0 0.0 -1.57079632679"/>
-        <!-- <origin xyz="-0.27 0.0 -0.0" rpy="0.0 0.0 -1.57079632679"/> -->
+        <!-- <origin xyz="-0.27 0.0 -0.038" rpy="0.0 0.0 -1.57079632679"/> -->
+        <origin xyz="-0.27 0.0 -0.0" rpy="0.0 0.0 -1.57079632679"/>
         <parent link="base_link"/>
         <child link="sway_thruster_link"/>

File: oasis_auv_stonefish/description/oasis_auv.scn.xacro (robot description, xacro)
@@ -13,16 +13,16 @@
         <robot name="${robot_name}" fixed="false" self_collisions="false">
             <base_link name="Vehicle" type="compound" physics="submerged">
-                <external_part name="Hull" type="model" physics="submerged" buoyant="true">
+                <external_part name="Hull" type="model" physics="submerged" buoyant="false">
                     <physical>
-                        <mesh filename="body.obj" scale="1.0"/>
+                        <mesh filename="oasis_body.obj" scale="0.001"/>
                         <origin rpy="0.0 -1.571 1.571" xyz="0.0 0.0 0.0"/>
                     </physical>
                     <visual>
-                        <mesh filename="body.obj" scale="1.0"/>
+                        <mesh filename="oasis_body.obj" scale="0.001"/>
                         <origin rpy="0.0 -1.571 1.571" xyz="0.0 0.0 0.0"/>
                     </visual>
                     <material name="Neutral"/>
                     <look name="yellow"/>
-                    <mass value="30"/>
+                    <mass value="0.5"/>
                     <!-- <inertia xyz="1.0 10.0 10.0"/> -->
                     <compound_transform rpy="0.0 0.0 0.0" xyz="0.0 0.0 0.0"/>
@@ -30,4 +30,14 @@
                     <cg xyz="0.565 0.0 0.00" rpy="0.0 0.0 0.0"/>
                 </external_part>
+                <internal_part name="lumsum_body" type="cylinder" physics="surface" buoyant="true">
+                    <dimensions radius="0.08" height="1.22"/>
+                    <origin rpy="0.0 -1.571 0.0" xyz="0.5 0.0 0.0"/>
+                    <material name="Neutral"/>
+                    <mass value="21.0"/>
+                    <look name="grey"/>
+                    <!-- <compound_transform rpy= "0.0 0.0 0.0" xyz="0.9 0 0.057"/> -->
+                    <!-- <compound_transform rpy= "0.0 0.0 0.0" xyz="0.847 0 0.057"/> -->
+                    <compound_transform rpy= "0.0 0.0 0.0" xyz="0.0 0 0.0"/>
+                </internal_part>
                 <internal_part name="Foam" type="box" physics="surface" buoyant="true">
                     <dimensions xyz="0.23 0.058 0.042"/>
@@ -37,5 +47,6 @@
                     <look name="grey"/>
                     <!-- <compound_transform rpy= "0.0 0.0 0.0" xyz="0.9 0 0.057"/> -->
-                    <compound_transform rpy= "0.0 0.0 0.0" xyz="0.847 0 0.057"/>
+                    <!-- <compound_transform rpy= "0.0 0.0 0.0" xyz="0.847 0 0.057"/> -->
+                    <compound_transform rpy= "0.0 0.0 0.0" xyz="0.5 0 0.057"/>
                     <!-- <compound_transform rpy= "0.0 0.0 0.0" xyz="0.347 0 0.057"/> -->
                 </internal_part>
@@ -90,4 +101,15 @@
                 <ros_subscriber topic="/${robot_name}/control/thruster/heave_bow"/>
             </actuator>
+            <actuator name="ThrusterHeaveStern" type="thruster">
+                <link name="Base"/>
+                <origin rpy="0.0 -1.571 0.0" xyz="0.2074 0.0 0.03"/>
+                <specs thrust_coeff="0.4315" thrust_coeff_backward="0.3404" torque_coeff="0.01" max_rpm="3000.0"/>
+                <propeller diameter="0.08" right="true">
+                    <mesh filename="prop.obj" scale="1.0"/>
+                    <material name="Delrin"/>
+                    <look name="white"/>
+                </propeller>
+                <ros_subscriber topic="/${robot_name}/control/thruster/heave_stern"/>
+            </actuator>
             <actuator name="ThrusterSurge" type="thruster">
                 <link name="Base"/>
@@ -122,10 +144,10 @@
                 <ros_publisher topic="/${robot_name}/imu/stonefish/data"/>
             </sensor>
-            <!-- <sensor name="gps" type="gps" rate="1.0">
+            <sensor name="gps" type="gps" rate="1.0">
                 <link name="Base"/>
-                <origin rpy="0.0 0.0 0.0" xyz="-0.7 0.0 -0.3"/>
+                <origin rpy="0.0 0.0 0.0" xyz="0.0 0.0 -0.3"/>
                 <noise ned_position="0.1"/>
                 <ros_publisher topic="/${robot_name}/gps/fix"/>
-            </sensor> -->
+            </sensor>
             <sensor name="Cam" rate="5.0" type="camera">
                 <link name="Base"/>

File: oasis_auv_stonefish/scenarios/under_ice.scn.xacro (robot description, xacro)
@@ -10,5 +10,5 @@
     <xacro:arg name="robot_name" default="changeme"/>
     <xacro:include filename="$(find oasis_auv_stonefish)/description/oasis_auv.scn.xacro"/>
-    <xacro:oasis_auv robot_name="$(arg robot_name)" xyz="0.0 0.0 5.0" rpy="0.0 0.0 0.0"/>
+    <xacro:oasis_auv robot_name="$(arg robot_name)" xyz="0.0 0.0 0.0" rpy="0.0 0.0 0.0"/>
     <environment>
         <ned latitude="41" longitude="-71"/>
@@ -27,5 +27,5 @@
         </ocean>
         <atmosphere>
-            <sun azimuth="50.0" elevation="30.0"/>
+            <sun azimuth="50.0" elevation="70.0"/>
         </atmosphere>
     </environment>

Commit message: tuned PID for auv mode

File: oasis_auv_description/urdf/base_sf.urdf.xacro (robot description, xacro)
@@ -29,5 +29,5 @@
     <link name="dvl"/>
     <joint name="dvl_joint" type="fixed">
-        <origin xyz="-0.3 0.0 0.092" rpy="0.0 0.0 0.0"/>
+        <origin xyz="-0.3 0.0 0.092" rpy="3.1415926 0.0 0.0"/>
         <parent link="base_link"/>
         <child link="dvl"/>
@@ -35,5 +35,5 @@
      <link name="dvl_sf"/>
     <joint name="dvl_sf_joint" type="fixed">
-        <origin xyz="-0.3 0.0 0.092" rpy="3.1415926 0.0 0.0"/>
+        <origin xyz="-0.3 0.0 0.092" rpy="0.0 0.0 0.0"/>
         <parent link="base_link"/>
         <child link="dvl_sf"/>

File: oasis_auv_stonefish/description/oasis_auv.scn.xacro (robot description, xacro)
@@ -53,7 +53,7 @@
                     <look name="yellow"/>
                     <!-- forward position -->
-                    <!-- <compound_transform rpy= "0.0 0.0 0.0" xyz="0.847 0 0.057"/> -->
+                    <compound_transform rpy= "0.0 0.0 0.0" xyz="0.847 0 0.057"/>
                     <!-- backward position -->
-                    <compound_transform rpy= "0.0 0.0 0.0" xyz="0.347 0 0.057"/>
+                    <!-- <compound_transform rpy= "0.0 0.0 0.0" xyz="0.347 0 0.057"/> -->
                 </internal_part>
                 <external_part name="ThrusterDuctSurge" type="model" physics="surface" buoyant="true">
@@ -138,5 +138,5 @@
             <sensor name="dvl_sf" type="dvl" rate="5.0">
                 <link name="Base"/>
-                <origin rpy="0.0 0.0 0.0" xyz="0.1 0.0 -0.092"/>
+                <origin rpy="3.1415926 0.0 0.0" xyz="0.1 0.0 -0.092"/>
                 <specs beam_angle="30.0"/>
                 <range velocity="9.0 9.0 9.0" altitude_min="0.2" altitude_max="200.0"/>

File: oasis_auv_stonefish/scenarios/under_ice.scn.xacro (robot description, xacro)
@@ -43,3 +43,16 @@
         <world_transform xyz="0.0 0.0 0.0" rpy="0.0 0.0 0.0"/>
     </static> -->
+    <static name="Bottom" type="model">
+        <physical>
+            <mesh filename="flat_terrain.obj" scale="2.0" convex="true"/>
+            <origin xyz="0.0 0.0 0.0" rpy="0.0 0.0 0.0"/>
+        </physical>
+        <visual>
+            <mesh filename="flat_terrain.obj" scale="2.0"/>
+            <origin xyz="0.0 0.0 0.0" rpy="0.0 0.0 0.0"/>
+        </visual>
+        <material name="Rock"/>
+        <look name="Gray"/>
+        <world_transform xyz="0.0 0.0 40.0" rpy="0.0 0.0 0.0"/>
+    </static>
 </scenario>

Commit message: servo joint working in simulation and rviz

File: oasis_auv_description/urdf/base_sf.urdf.xacro (robot description, xacro)
@@ -52,9 +52,19 @@
     </joint>
     <!-- thrusters -->
-    <link name="surge_thruster_link"/>
-    <joint name="surge_thruster_joint" type="fixed">
+    <link name="surge_servo_link"/>
+    <joint name="surge_servo_joint" type="fixed">
         <origin xyz="-0.5 0.0 0.0" rpy="0.0 0.0 0.0"/>
         <parent link="base_link"/>
+        <child link="surge_servo_link"/>
+    </joint>
+    <link name="surge_thruster_link"/>
+    <joint name="oasis_auv/servo_joint" type="revolute">
+        <origin xyz="0.0 0.0 0.0" rpy="0.0 0.0 0.0"/>
+        <axis xyz="0.0 0.0 1.0"/>
+        <parent link="surge_servo_link"/>
         <child link="surge_thruster_link"/>
+        <!-- <calibration rising="0.0"/> -->
+        <!-- <dynamics damping="0.0" friction="0.0"/> -->
+        <limit effort="10" velocity="1.0" lower="-1.0" upper="1.01" />
     </joint>
     <link name="heave_bow_thruster_link"/>

File: oasis_auv_stonefish/description/oasis_auv.scn.xacro (robot description, xacro)
@@ -118,6 +118,24 @@
                 <ros_subscriber topic="/${robot_name}/control/thruster/heave_stern"/>
             </actuator>
+            <link name="surge_servo_link" type="box" physics="submerged"  buoyant="false">
+                <dimensions xyz="0.0001 0.0002 0.00001"/>
+                <origin xyz="-0.2 0.0 0.0" rpy="0.0 0.0 0.0"/>
+                <material name="Neutral"/>
+                <look name="Green"/>
+            </link>
+            <joint name="servo_joint" type="revolute">
+                <parent name="Base"/>
+                <child name="surge_servo_link"/>
+                <origin xyz="0.0 0.0 0.0" rpy="0.0 0.0 0.0"/>
+                <axis xyz="0.0 0.0 1.0"/>
+            </joint>
+            <actuator name="surge_servo" type="servo">
+                <joint name="servo_joint"/>
+                <controller position_gain="1.1" velocity_gain="0.1" max_torque="10.0"/>
+                <initial position="-0.5"/>
+                <ros_subscriber topic="/${robot_name}/control/servo/surge"/>
+            </actuator>
             <actuator name="ThrusterSurge" type="thruster">
-                <link name="Base"/>
+                <link name="surge_servo_link"/>
                 <origin rpy="0.0 0.0 0.0" xyz="-0.2 0.0 0.0"/>
                 <specs thrust_coeff="1.7568" thrust_coeff_backward="1.0882" torque_coeff="0.01" max_rpm="3000.0"/>
@@ -161,6 +179,8 @@
                 <origin xyz="1.25 0.0 0.05" rpy="0.0 1.571 0.0"/>
                 <ros_publisher topic="/${robot_name}/camera/data"/>
-            </sensor>
+            </sensor>    <initial position="0.5"/>
             <world_transform rpy="${rpy}" xyz="${xyz}"/>
+            <ros_publisher servos="/${robot_name}/control/servos/joint_states"/>
+            <ros_subscriber servos="/${robot_name}/control/servos/desired_joint_states"/>
         </robot>
     </xacro:macro>
